Commit message: checkpoint

File: src/go2_robot/urdf/go2.urdf (robot description, URDF)
Before this commit: robot go2, 31 links, 30 joints
Links:
- added link map
- added link odom
Joints:
- added joint map_joint: type fixed, parent map, child odom, origin xyz=0 0 0 rpy=0 0 0
- added joint odom_joint: type fixed, parent odom, child base_link, origin xyz=0 0 0 rpy=0 0 0

File: src/go2_robot/urdf/go2_on_steroids.urdf (robot description, URDF)
Before this commit: robot go2, 33 links, 32 joints
Links:
- link FL_calf: geometry collision cylinder length=0.12 radius=0.012; visual mesh filename=package://go2_robot/dae/calf.dae
- link FL_foot: geometry collision sphere radius=0.022; visual mesh filename=package://go2_robot/dae/foot.dae
- link FL_hip: geometry collision cylinder length=0.04 radius=0.046; visual mesh filename=package://go2_robot/dae/hip.dae
- link FL_thigh: geometry collision box size=0.213 0.0245 0.034; visual mesh filename=package://go2_robot/dae/thigh.dae
- link FR_calf: geometry collision cylinder length=0.12 radius=0.013; visual mesh filename=package://go2_robot/dae/calf_mirror.dae
- link FR_foot: geometry collision sphere radius=0.022; visual mesh filename=package://go2_robot/dae/foot.dae
- link FR_hip: geometry collision cylinder length=0.04 radius=0.046; visual mesh filename=package://go2_robot/dae/hip.dae
- link FR_thigh: geometry collision box size=0.213 0.0245 0.034; visual mesh filename=package://go2_robot/dae/thigh_mirror.dae
- link RL_calf: geometry collision cylinder length=0.12 radius=0.013; visual mesh filename=package://go2_robot/dae/calf.dae
- link RL_foot: geometry collision sphere radius=0.022; visual mesh filename=package://go2_robot/dae/foot.dae
- link RL_hip: geometry collision cylinder length=0.04 radius=0.046; visual mesh filename=package://go2_robot/dae/hip.dae
- link RL_thigh: geometry collision box size=0.213 0.0245 0.034; visual mesh filename=package://go2_robot/dae/thigh.dae
- link RR_calf: geometry collision cylinder length=0.12 radius=0.013; visual mesh filename=package://go2_robot/dae/calf_mirror.dae
- link RR_foot: geometry collision sphere radius=0.022; visual mesh filename=package://go2_robot/dae/foot.dae
- link RR_hip: geometry collision cylinder length=0.04 radius=0.046; visual mesh filename=package://go2_robot/dae/hip.dae
- link RR_thigh: geometry collision box size=0.213 0.0245 0.034; visual mesh filename=package://go2_robot/dae/thigh_mirror.dae
- link base_link: geometry collision box size=0.3762 0.0935 0.114; visual mesh filename=package://go2_robot/meshes/base_link.STL
- link front_d_camera: geometry collision mesh filename=package://go2_robot/meshes/front_d_camera.STL; visual mesh filename=package://go2_robot/meshes/front_d_camera.STL
- link left_d_camera: geometry collision mesh filename=package://go2_robot/meshes/left_d_camera.STL; visual mesh filename=package://go2_robot/meshes/left_d_camera.STL
- link lidar: geometry collision mesh filename=package://go2_robot/meshes/lidar_link.STL; visual mesh filename=package://go2_robot/meshes/lidar_link.STL
- link right_d_camera: geometry collision mesh filename=package://go2_robot/meshes/right_d_camera.STL; visual mesh filename=package://go2_robot/meshes/right_d_camera.STL

File: src/go2_robot/urdf/go2_with_realsense.urdf (robot description, URDF)
Before this commit: robot go2, 35 links, 34 joints
Links:
- link FL_calf: geometry collision cylinder length=0.12 radius=0.012; visual mesh filename=package://go2_robot/dae/calf.dae
- link FL_foot: geometry collision sphere radius=0.022; visual mesh filename=package://go2_robot/dae/foot.dae
- link FL_hip: geometry collision cylinder length=0.04 radius=0.046; visual mesh filename=package://go2_robot/dae/hip.dae
- link FL_thigh: geometry collision box size=0.213 0.0245 0.034; visual mesh filename=package://go2_robot/dae/thigh.dae
- link FR_calf: geometry collision cylinder length=0.12 radius=0.013; visual mesh filename=package://go2_robot/dae/calf_mirror.dae
- link FR_foot: geometry collision sphere radius=0.022; visual mesh filename=package://go2_robot/dae/foot.dae
- link FR_hip: geometry collision cylinder length=0.04 radius=0.046; visual mesh filename=package://go2_robot/dae/hip.dae
- link FR_thigh: geometry collision box size=0.213 0.0245 0.034; visual mesh filename=package://go2_robot/dae/thigh_mirror.dae
- link RL_calf: geometry collision cylinder length=0.12 radius=0.013; visual mesh filename=package://go2_robot/dae/calf.dae
- link RL_foot: geometry collision sphere radius=0.022; visual mesh filename=package://go2_robot/dae/foot.dae
- link RL_hip: geometry collision cylinder length=0.04 radius=0.046; visual mesh filename=package://go2_robot/dae/hip.dae
- link RL_thigh: geometry collision box size=0.213 0.0245 0.034; visual mesh filename=package://go2_robot/dae/thigh.dae
- link RR_calf: geometry collision cylinder length=0.12 radius=0.013; visual mesh filename=package://go2_robot/dae/calf_mirror.dae
- link RR_foot: geometry collision sphere radius=0.022; visual mesh filename=package://go2_robot/dae/foot.dae
- link RR_hip: geometry collision cylinder length=0.04 radius=0.046; visual mesh filename=package://go2_robot/dae/hip.dae
- link RR_thigh: geometry collision box size=0.213 0.0245 0.034; visual mesh filename=package://go2_robot/dae/thigh_mirror.dae
- link base_link: geometry collision box size=0.3762 0.0935 0.114; visual mesh filename=package://go2_robot/dae/base.dae

Commit message: URDF visualization completed by jhyoon

File: src/go2_robot/urdf/go2.urdf (robot description, URDF)
Before this commit: robot go2, 33 links, 32 joints
Links:
- link FL_calf: geometry collision cylinder length=0.12 radius=0.012; visual mesh filename=package://go2_robot/dae/calf.dae
- link FL_foot: geometry collision sphere radius=0.022; visual mesh filename=package://go2_robot/dae/foot.dae
- link FL_hip: geometry collision cylinder length=0.04 radius=0.046; visual mesh filename=package://go2_robot/dae/hip.dae
- link FL_thigh: geometry collision box size=0.213 0.0245 0.034; visual mesh filename=package://go2_robot/dae/thigh.dae
- link FR_calf: geometry collision cylinder length=0.12 radius=0.013; visual mesh filename=package://go2_robot/dae/calf_mirror.dae
- link FR_foot: geometry collision sphere radius=0.022; visual mesh filename=package://go2_robot/dae/foot.dae
- link FR_hip: geometry collision cylinder length=0.04 radius=0.046; visual mesh filename=package://go2_robot/dae/hip.dae
- link FR_thigh: geometry collision box size=0.213 0.0245 0.034; visual mesh filename=package://go2_robot/dae/thigh_mirror.dae
- link RL_calf: geometry collision cylinder length=0.12 radius=0.013; visual mesh filename=package://go2_robot/dae/calf.dae
- link RL_foot: geometry collision sphere radius=0.022; visual mesh filename=package://go2_robot/dae/foot.dae
- link RL_hip: geometry collision cylinder length=0.04 radius=0.046; visual mesh filename=package://go2_robot/dae/hip.dae
- link RL_thigh: geometry collision box size=0.213 0.0245 0.034; visual mesh filename=package://go2_robot/dae/thigh.dae
- link RR_calf: geometry collision cylinder length=0.12 radius=0.013; visual mesh filename=package://go2_robot/dae/calf_mirror.dae
- link RR_foot: geometry collision sphere radius=0.022; visual mesh filename=package://go2_robot/dae/foot.dae
- link RR_hip: geometry collision cylinder length=0.04 radius=0.046; visual mesh filename=package://go2_robot/dae/hip.dae
- link RR_thigh: geometry collision box size=0.213 0.0245 0.034; visual mesh filename=package://go2_robot/dae/thigh_mirror.dae
- link base_link: geometry collision box size=0.3762 0.0935 0.114; visual mesh filename=package://go2_robot/dae/base.dae

Commit message: marker and yolo clear

File: src/go2_robot/urdf/go2.urdf (robot description, URDF)
Before this commit: robot go2, 31 links, 30 joints
Links:
- added link front_realsense_camera_link, mass 0.094; collision box size=0.025 0.09 0.025; visual box size=0.025 0.09 0.025
- added link yujin_lidar, mass 0.001; visual cylinder length=0.05 radius=0.03
Joints:
- added joint front_camera_to_front_realsense_joint: type fixed, parent front_camera, child front_realsense_camera_link, origin xyz=-0.02909936 -0.06333103 0.00976318 rpy=0.04475 -0.03469 -0.00758, axis 0 0 0
- added joint yujin_lidar_joint: type fixed, parent base_link, child yujin_lidar, origin xyz=-0.124017 0 0.30050 rpy=0 0 3.3

Commit message: arudo marker function clear

File: src/go2_robot/urdf/go2.urdf (robot description, URDF)
Before this commit: robot go2, 33 links, 32 joints
Joints:
- joint front_camera_to_front_realsense_joint: origin xyz=-0.02909936 -0.06333103 0.00976318 rpy=0.04475 -0.03469 -0.00758 -> xyz=-0.08 0.0 0.00976318 rpy=0.04475 -0.03469 -0.00758
